File: SandKrux.kicad_sch (KiCad schematic)
At the start: 67 parts, among them CN1 527450697, J1 FH12-40S-0.5SH_55_, U1 K210_C913414, U2 AXP173, U3 MT9700-N, U4 XC6206P182MR_C347373, U5 GD25LQ128EWIGR, U6 TMI7003C, U7 SGM803-TXN3/TR_C5152602, U8 XC6206P302MR_C347375, X1 X322526MMB4SI

Commit message: LCD E CAP_TOUTCH E JLC DOWNLOADER
Parts:
- removed J1: FH12-40S-0.5SH_55_, KiCad:FH1240S05SH55, symbol FH12-40S-0_5SH_55_:FH12-40S-0.5SH_55_
- added C37, C50: 10uF, Capacitor_SMD:C_0201_0603Metric, symbol Device:C
- added C38, C49: 100nF, Capacitor_SMD:C_0201_0603Metric, symbol Device:C
- added C39, C40, C41, C42, C43, C44, C45, C46, C47, C48: 100pF, Capacitor_SMD:C_0201_0603Metric, symbol Device:C
- added FPC3: FH12-40S-0.5SH(55), easyeda2kicad:FPC-SMD_FH12-40S-0.5SH-55, symbol easyeda2kicad:FH12-40S-0.5SH(55)
- added FPC4: FH12-6S-0.5SH(55), easyeda2kicad:FPC-SMD_FH12-6S-0.5SH-55, symbol easyeda2kicad:FH12-6S-0.5SH(55)
- added J1: Conn_01x02, Connector_PinHeader_2.54mm:PinHeader_1x02_P2.54mm_Vertical, symbol Connector_Generic:Conn_01x02
- added Q1: S8050, PCM_JLCPCB:Q_SOT-23, symbol PCM_JLCPCB-Transistors:NPN,S8050
- added Q2: SI2301CDS-T1-GE3, PCM_JLCPCB:Q_SOT-89, symbol PCM_JLCPCB-Transistors:PMOS,SI2301CDS-T1-GE3
- added R12: 5.1R, Resistor_SMD:R_0201_0603Metric, symbol Device:R
- added R13, R14: 100R, Resistor_SMD:R_0201_0603Metric, symbol Device:R
- added R15, R16, R17: 10K, Resistor_SMD:R_0201_0603Metric, symbol Device:R
- added R18, R21: 0R, Resistor_SMD:R_0201_0603Metric, symbol Device:R
- added R19, R20, R22, R23, R27: NC, Resistor_SMD:R_0201_0603Metric, symbol Device:R
- added R24, R25, R26: 5.1K, Resistor_SMD:R_0201_0603Metric, symbol Device:R
Connections:
- net GND: now also C37.2, C38.2, C39.2, C40.2, C41.2, C42.2, C43.2, C44.2, C45.2, C46.2, C47.2, C48.2, C49.2, C50.2, FPC3.16, FPC3.34, FPC3.35, FPC3.36, FPC3.37, FPC3.41 (MH1), FPC3.42 (MH2), FPC3.5, FPC4.6, FPC4.7, FPC4.8, Q1.2 (E), R16.1, R18.2, R19.2, R22.2, R23.2, R24.2
- net LCD_CS: now also FPC3.9
- net LCD_DC: now also C48.1, FPC3.10
- net LCD_RST: now also FPC3.15, R13.1
- net LCD_WR: now also C47.1, FPC3.11
- net at C4.2, C5.2, C6.2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: now also C37.1, C49.1, C50.1, FPC4.1, Q2.2 (S), R15.2, R17.1
- new net: Q1.1 (B), R13.2, R16.2
- new net: Q1.3 (C), R14.1, R15.1
- new net: Q2.1 (G), R14.2
- new net: FPC3.33, R12.1
- new net CAPTOUCH_RST: C38.1, FPC4.5, J1.1 (Pin_1), R17.2
- new net FUNCTION2: FPC4.4, J1.2 (Pin_2)
- new net I2C_SCL: FPC4.3
- new net I2C_SDA: FPC4.2
- new net IM0: FPC3.38, R22.1, R25.1
- new net IM1: FPC3.39, R23.1, R26.1
- new net IM2: FPC3.40, R24.1, R27.1
- new net LCD_BACKLIGHT: Q2.3 (D), R12.2
- new net LCD_D0: C39.1, FPC3.17
- new net LCD_D1: C40.1, FPC3.18
- new net LCD_D2: C41.1, FPC3.19
- new net LCD_D3: C42.1, FPC3.20
- new net LCD_D4: C43.1, FPC3.21
- new net LCD_D5: C44.1, FPC3.22
- new net LCD_D6: C45.1, FPC3.23
- new net LCD_D7: C46.1, FPC3.24
- new net VCC_1V83V3: FPC3.12, R20.2, R21.2, R25.2, R26.2, R27.2
- new net VCC_6: R18.1, R20.1
- new net VCC_7: R19.1, R21.1
- no-connect marks 55 -> 70
Other:
- note added: "LCD E CAP_TOUTCH"
- moved on the sheet: CN1, U2, U3
