File: untitled.kicad_sch (KiCad schematic)
At the start: 63 parts, among them U1 K210_C913414, U4 XC6206P182MR_C347373, U5 GD25LQ128EWIGR, U6 TMI7003C, U7 SGM803-TXN3/TR_C5152602, U8 XC6206P302MR_C347375, X1 X322526MMB4SI

Commit message: NGFF 67p conector no esquematico
Parts:
- added U12: PCIE-67P42H, easyeda2kicad:PCIE-SMD_75P-P0.50_HYC01B-05NGFF-420, symbol easyeda2kicad:PCIE-67P42H
Connections:
- net 1V8: now also U12.75
- net 5v: now also U12.2, U12.4
- net BOOT: now also U12.53
- net DVP_D0: now also U12.60
- net DVP_D1: now also U12.62
- net DVP_D2: now also U12.64
- net DVP_D3: now also U12.66
- net DVP_D4: now also U12.68
- net DVP_D5: now also U12.70
- net DVP_D6: now also U12.72
- net DVP_D7: now also U12.74
- net DVP_HSYNC: now also U12.22
- net DVP_PCLK: now also U12.20
- net DVP_PWDN: now also U12.32
- net DVP_RST: now also U12.30
- net DVP_SCL: now also U12.26
- net DVP_SDA: now also U12.28
- net DVP_VSYNC: now also U12.24
- net DVP_XCLK: now also U12.34
- net GND: now also U12.6, U12.8
- net IO_10: now also U12.65
- net IO_11: now also U12.67
- net IO_12: now also U12.61
- net IO_13: now also U12.63
- net IO_14: now also U12.57
- net IO_15: now also U12.59
- net IO_17: now also U12.55
- net IO_21: now also U12.47
- net IO_22: now also U12.41
- net IO_23: now also U12.43
- net IO_24: now also U12.37
- net IO_25: now also U12.39
- net IO_26: now also U12.33
- net IO_27: now also U12.35
- net IO_28: now also U12.29
- net IO_29: now also U12.31
- net IO_30: now also U12.25
- net IO_31: now also U12.27
- net IO_32: now also U12.21
- net IO_33: now also U12.23
- net IO_34: now also U12.9
- net IO_35: now also U12.11
- net IO_4: now also U12.42
- net IO_5: now also U12.40
- net IO_6: now also U12.38
- net IO_7: now also U12.71
- net IO_8: now also U12.36
- net IO_9: now also U12.69
- net RST: now also U12.10
- net SPI0_D0: now also U12.58
- net SPI0_D1: now also U12.56
- net SPI0_D2: now also U12.54
- net SPI0_D3: now also U12.52
- net SPI0_D4: now also U12.50
- net SPI0_D5: now also U12.48
- net SPI0_D7: now also U12.44
- net at C4.2, C5.2, C6.2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: now also U12.73
- new net IO_36: U12.7
- new net IO_37: U12.3
- new net IO_38: U12.5
- new net IO_39: U12.1
- new net MIC_BCK: U12.49
- new net MIC_DAT3: U12.45
- new net MIC_WS: U12.51
- new net SPI0_D6: U12.46
- no-connect marks 55 -> 1
