File: SandKrux.kicad_pcb (KiCad board)
At the start: 2 copper layers, 58.3 x 98.2 mm, 169 parts, among them CN2 1.25mm-2P socket, IC1 TROPIC01_chip, Q1 S8050, Q2 SI2301CDS-T1-GE3, SW1 TL3330AF130QG, SW2 TL3330AF130QG, SW3 TL3330AF130QG, SW4 TL3330AF130QG, SW5 TL3330AF130QG, U1 K210_C913414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

Commit message: correcao de erros nas vias
Parts:
- added Sign_OSHW_7.3x6.0mm: Sign_OSHW_7.3x6.0mm, OLIMEX_Signs-FP:Sign_OSHW_7.3x6.0mmn, F.Cu at (126.8, 183.6)
- moved REF** 5.95 mm to (127.2, 173.8)
- moved SW1 1.43 mm to (82.1, 153.2)
- moved SW2 1.43 mm to (82.1, 162.7)
- moved SW5 0.92 mm to (82.6, 120.2)
- moved SW3 0.91 mm to (82.6, 101.6)
- moved R39 0.91 mm to (85.6, 109.9)
- moved SW4 0.91 mm to (82.6, 110.9)
- moved H3 0.73 mm to (84.2, 182.9)
- moved R40 0.71 mm to (85.4, 119.7)
- moved R38 0.71 mm to (85.4, 99.6)
- moved R41 0.71 mm to (85.4, 120.5)
- moved H2 0.62 mm to (84.2, 92.7)
- moved H4 0.52 mm to (134.5, 182.9)
- moved H1 0.35 mm to (134.5, 92.7)
- moved R21 0.22 mm to (121.0, 142.6)
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Routing:
- net GND: track 486.5 -> 466.9 mm, vias 150 -> 148
- net /3V3: track 219.1 -> 214.5 mm
- net /KEY2: track 56.6 -> 55.3 mm
- net /RST: track 78.9 -> 80.2 mm
- net /KEY1: track 68.2 -> 67.1 mm
